File: DCC.kicad_sch (KiCad schematic)
At the start: 6 parts, among them J1 Screw_Terminal_01x02, U3 6N137

Commit message: finalized default template
Parts:
- D1: footprint Diode_SMD:D_SMA_Handsoldering -> Diode_SMD:D_SOD-323; JLCPCB Part# (none) -> C2128
Connections:
- net DCC_A: now also J1.1 (Pin_1); no longer J1.2 (Pin_2)
- net DCC_B: now also J1.2 (Pin_2); no longer J1.1 (Pin_1)
Other:
- moved on the sheet: J1
Changed lines of the file:
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@@
 (kicad_sch (version 20211123) (generator eeschema)
   (paper "A4")
-  (junction (at 113.03 95.25) (diameter 0) (color 0 0 0 0)
+  (junction (at 115.57 102.87) (diameter 0) (color 0 0 0 0)
   )
   (junction (at 151.13 96.52) (diameter 0) (color 0 0 0 0)
   )
+  (junction (at 115.57 95.25) (diameter 0) (color 0 0 0 0)
+  )
   (junction (at 151.13 86.36) (diameter 0) (color 0 0 0 0)
   )
   (junction (at 143.51 86.36) (diameter 0) (color 0 0 0 0)
   )
-  (junction (at 113.03 102.87) (diameter 0) (color 0 0 0 0)
-  )
   (wire (pts (xy 135.89 101.6) (xy 135.89 107.95))
     (stroke (width 0) (type default) (color 0 0 0 0))
@@
     (stroke (width 0) (type default) (color 0 0 0 0))
   )
-  (wire (pts (xy 113.03 95.25) (xy 120.65 95.25))
-    (stroke (width 0) (type default) (color 0 0 0 0))
-  )
-  (wire (pts (xy 97.79 102.87) (xy 113.03 102.87))
-    (stroke (width 0) (type default) (color 0 0 0 0))
-  )
   (wire (pts (xy 97.79 95.25) (xy 97.79 97.79))
     (stroke (width 0) (type default) (color 0 0 0 0))
@@
     (stroke (width 0) (type default) (color 0 0 0 0))
   )
-  (wire (pts (xy 113.03 102.87) (xy 119.38 102.87))
+  (wire (pts (xy 115.57 95.25) (xy 120.65 95.25))
+    (stroke (width 0) (type default) (color 0 0 0 0))
+  )
+  (wire (pts (xy 115.57 102.87) (xy 119.38 102.87))
     (stroke (width 0) (type default) (color 0 0 0 0))
   )
@@
     (stroke (width 0) (type default) (color 0 0 0 0))
   )
+  (wire (pts (xy 97.79 102.87) (xy 115.57 102.87))
+    (stroke (width 0) (type default) (color 0 0 0 0))
+  )
   (wire (pts (xy 120.65 96.52) (xy 120.65 95.25))
     (stroke (width 0) (type default) (color 0 0 0 0))
@@
     (stroke (width 0) (type default) (color 0 0 0 0))
   )
-  (wire (pts (xy 109.22 95.25) (xy 113.03 95.25))
+  (wire (pts (xy 109.22 95.25) (xy 115.57 95.25))
     (stroke (width 0) (type default) (color 0 0 0 0))
   )
@@
     (pin "1")
   )
-  (symbol (lib_id "Connector:Screw_Terminal_01x02") (at 92.71 100.33 180) (unit 1)
-    (in_bom yes) (on_board yes) (fields_autoplaced)
-    (property "Reference" "J1" (id 0) (at 92.71 93.98 0))
-    (property "Value" "Screw_Terminal_01x02" (id 1) (at 92.71 93.98 0)
-      (effects (font (size 1.27 1.27)) hide)
-    )
-    (property "Footprint" "TerminalBlock_Phoenix:TerminalBlock_Phoenix_MKDS-1,5-2-5.08_1x02_P5.08mm_Horizontal" (id 2) (at 92.71 100.33 0)
-      (effects (font (size 1.27 1.27)) hide)
-    )
-    (property "Datasheet" "~" (id 3) (at 92.71 100.33 0)
+  (symbol (lib_id "Connector:Screw_Terminal_01x02") (at 92.71 97.79 0) (mirror y) (unit 1)
+    (in_bom yes) (on_board yes) (fields_autoplaced)
+    (property "Reference" "J1" (id 0) (at 92.71 95.3572 0))
+    (property "Value" "Screw_Terminal_01x02" (id 1) (at 92.71 104.14 0)
+      (effects (font (size 1.27 1.27)) hide)
+    )
+    (property "Footprint" "TerminalBlock_Phoenix:TerminalBlock_Phoenix_MKDS-1,5-2-5.08_1x02_P5.08mm_Horizontal" (id 2) (at 92.71 97.79 0)
+      (effects (font (size 1.27 1.27)) hide)
+    )
+    (property "Datasheet" "~" (id 3) (at 92.71 97.79 0)
       (effects (font (size 1.27 1.27)) hide)
     )
@@
     )
     (property "JLCPCB Part#" "C17513" (id 4) (at 105.41 95.25 0)
-      (effects (font (size 1.27 1.27)) hide)
-    )
-    (pin "1")
-    (pin "2")
-  )
-  (symbol (lib_id "Device:D") (at 113.03 99.06 270) (unit 1)
-    (in_bom yes) (on_board yes) (fields_autoplaced)
-    (property "Reference" "D1" (id 0) (at 115.062 98.2253 90)
-      (effects (font (size 1.27 1.27)) (justify left))
-    )
-    (property "Value" "D" (id 1) (at 115.062 100.7622 90)
-      (effects (font (size 1.27 1.27)) (justify left))
-    )
-    (property "Footprint" "Diode_SMD:D_SMA_Handsoldering" (id 2) (at 113.03 99.06 0)
-      (effects (font (size 1.27 1.27)) hide)
-    )
-    (property "Datasheet" "~" (id 3) (at 113.03 99.06 0)
       (effects (font (size 1.27 1.27)) hide)
     )
@@
     (pin "8")
   )
+  (symbol (lib_id "Device:D") (at 115.57 99.06 270) (unit 1)
+    (in_bom yes) (on_board yes)
+    (property "Reference" "D1" (id 0) (at 113.03 99.06 0))
+    (property "Value" "D" (id 1) (at 113.03 101.6 0)
+      (effects (font (size 1.27 1.27)) hide)
+    )
+    (property "Footprint" "Diode_SMD:D_SOD-323" (id 2) (at 115.57 99.06 0)
+      (effects (font (size 1.27 1.27)) hide)
+    )
+    (property "Datasheet" "~" (id 3) (at 115.57 99.06 0)
+      (effects (font (size 1.27 1.27)) hide)
+    )
+    (property "JLCPCB Part#" "C2128" (id 4) (at 115.57 99.06 0)
+      (effects (font (size 1.27 1.27)) hide)
+    )
+    (pin "1")
+    (pin "2")
+  )
 )
