File: Lnet.kicad_sch (KiCad schematic)
At the start: 12 parts, among them J17 RJ12, J18 RJ12, Q1 BC847, U15 LM311

Commit message: finalized default template
Parts:
- removed D11, D12: D, Diode_SMD:D_SMA, symbol Device:D
- added D2, D3: D, Diode_SMD:D_SOD-323, symbol Device:D
- Q1: JLCPCB Part# (none) -> C181140
- R23: JLCPCB Part# (none) -> C17556
- R24: JLCPCB Part# (none) -> C17713
- R25: JLCPCB Part# (none) -> C17414
- R26: JLCPCB Part# (none) -> C17470
- R27: JLCPCB Part# (none) -> C17560
- R28: footprint Resistor_SMD:R_0805_2012Metric_Pad1.20x1.40mm_HandSolder -> Resistor_SMD:R_0603_1608Metric_Pad0.98x0.95mm_HandSolder; JLCPCB Part# (none) -> C21190
Connections:
- net railsyncA: now also D3.2 (A)
- net railsyncB: now also D2.2 (A)
- new net VCC: D2.1 (K), D3.1 (K)
