File: uController.kicad_sch (KiCad schematic)
At the start: 8 parts, among them SW1 SW_SPST, U1 ATmega328-A, U2 HEADER_3x2, Y1 crystal_arduino

Commit message: finalized default template
Parts:
- added C3: 100nF, Capacitor_SMD:C_0603_1608Metric_Pad1.08x0.95mm_HandSolder, symbol Device:C
- added D4: LED, LED_SMD:LED_0805_2012Metric_Pad1.15x1.40mm_HandSolder, symbol Device:LED
- added R6: 6k2, Resistor_SMD:R_0603_1608Metric_Pad0.98x0.95mm_HandSolder, symbol Device:R
Connections:
- net servo2 is gone; now on net Lnet_Tx: U1.13 (PB1)
- net servo3 is gone; now on net Lnet_Rx: U1.12 (PB0)
- net +5V: now also C3.2, R6.1
- net GND: now also C3.1
- net GPIO8: now reaches U1.1 (PD3)
- net TYPE: now reaches U1.19 (ADC6)
- net GPIO7: now reaches U1.2 (PD4)
- net GPIO13: now reaches U1.26 (PC3)
- net GPIO12: now reaches U1.27 (PC4)
- net GPIO11: now reaches U1.28 (PC5)
- net Rx renamed GPIO10
- net Tx renamed GPIO9
- net relay1 renamed GPIO5
- net relay2 renamed GPIO6
- net relay3 renamed LED
- net LED: now also D4.1 (K)
- net relay4 renamed GPIO16
- net relay5 renamed GPIO15
- net relay6 renamed GPIO14
- net servo1 renamed GPIO4
- net servo4 renamed GPIO1
- net servo5 renamed GPIO2
- net servo6 renamed GPIO3
- new net: D4.2 (A), R6.2
- no-connect marks 4 -> 1
Other:
- note added: "0"
- note added: "1"
- note added: "10"
- note added: "11"
- note added: "12"
- note added: "13"
- note added: "2"
- note added: "3"
- note added: "4"
- note added: "5"
- note added: "6"
- note added: "7"
- note added: "8"
- note added: "9"
- note added: "A0"
- note added: "A1"
- note added: "A2"
- note added: "A3"
- note added: "A4"
- note added: "A5"
